File: example_files/example.kicad_pcb (KiCad board)
At the start: 2 copper layers, 208 parts, among them K0 SW_SPST, K1 SW_SPST, K10 SW_SPST, K100 SW_SPST, K101 SW_SPST, K102 SW_SPST, K103 SW_SPST, K11 SW_SPST, K12 SW_SPST, K13 SW_SPST, K14 SW_SPST, K15 SW_SPST, K16 SW_SPST, K17 SW_SPST, K18 SW_SPST, K19 SW_SPST, K2 SW_SPST, K20 SW_SPST, K21 SW_SPST, K22 SW_SPST, K23 SW_SPST, K24 SW_SPST, K25 SW_SPST, K26 SW_SPST, K27 SW_SPST, K28 SW_SPST, K29 SW_SPST, K3 SW_SPST, K30 SW_SPST, K31 SW_SPST, K32 SW_SPST, K33 SW_SPST, K34 SW_SPST, K35 SW_SPST, K36 SW_SPST, K37 SW_SPST, K38 SW_SPST, K39 SW_SPST, K4 SW_SPST, K40 SW_SPST, K41 SW_SPST, K42 SW_SPST, K43 SW_SPST, K44 SW_SPST, K45 SW_SPST, K46 SW_SPST, K47 SW_SPST, K48 SW_SPST, K49 SW_SPST, K5 SW_SPST, K50 SW_SPST, K51 SW_SPST, K52 SW_SPST, K53 SW_SPST, K54 SW_SPST, K55 SW_SPST, K56 SW_SPST, K57 SW_SPST, K58 SW_SPST, K59 SW_SPST, K6 SW_SPST, K60 SW_SPST, K61 SW_SPST, K62 SW_SPST, K63 SW_SPST, K64 SW_SPST, K65 SW_SPST, K66 SW_SPST, K67 SW_SPST, K68 SW_SPST, K69 SW_SPST, K7 SW_SPST, K70 SW_SPST, K71 SW_SPST, K72 SW_SPST, K73 SW_SPST, K74 SW_SPST, K75 SW_SPST, K76 SW_SPST, K77 SW_SPST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

Commit message: Created a Makefile
Parts:
- removed D100, D101, D102, D103, D42, D43, D44, D45, D46, D47, D48, D49, D50, D51, D52, D53, D54, D55, D56, D57, D58, D59, D60, D61, D62, D63, D64, D65, D66, D67, D68, D69, D70, D71, D72, D73, D74, D75, D76, D77, D78, D79, D80, D81, D82, D83, D84, D85, D86, D87, D88, D89, D90, D91, D92, D93, D94, D95, D96, D97, D98, D99: D, Diode_THT:D_DO-35_SOD27_P7.62mm_Horizontal
- removed K100, K101, K102, K103, K42, K43, K44, K45, K46, K47, K48, K49, K50, K51, K52, K53, K54, K55, K56, K57, K58, K59, K60, K61, K62, K63, K64, K65, K66, K67, K68, K69, K70, K71, K72, K73, K74, K75, K76, K77, K78, K79, K80, K81, K82, K83, K84, K85, K86, K87, K88, K89, K90, K91, K92, K93, K94, K95, K96, K97, K98, K99: SW_SPST, Switch_Keyboard_Kailh:SW_Hotswap_Kailh_1.00u
- K0, K1, K10, K11, K12, K13, K14, K15, K16, K17, K18, K19, K2, K20, K21, K22, K23, K24, K25, K26, K27, K28, K29, K3, K30, K31, K32, K33, K34, K35, K36, K37, K38, K39, K4, K40, K41, K5, K6, K7, K8, K9: footprint Switch_Keyboard_Kailh:SW_Hotswap_Kailh_1.00u -> Switch_Keyboard_Cherry_MX:SW_Cherry_MX_PCB_1.00u
- moved D10 252.4 mm to (327.2, 80.7)
- moved D14 238.8 mm to (156.6, 181.4)
- moved D8 229.0 mm to (327.2, 105.5)
- moved D15 228.5 mm to (145.9, 185.0)
- moved D7 221.2 mm to (327.2, 102.0)
- moved D28 217.9 mm to (178.2, 181.4)
- moved D9 214.6 mm to (327.2, 109.1)
- moved D17 204.2 mm to (327.2, 84.2)
- moved D27 200.1 mm to (167.4, 185.0)
- moved K38 195.1 mm to (295.4, 109.1)
- moved D11 180.9 mm to (286.9, 161.3)
- moved D4 172.7 mm to (242.8, 181.4)
- moved K36 165.6 mm to (174.5, 89.0)
- moved D29 164.4 mm to (178.2, 185.0)
- moved D26 159.7 mm to (232.0, 188.5)
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
Commit message: Updated Makefile
Parts:
- added D42: D, Diode_THT:D_DO-35_SOD27_P7.62mm_Horizontal, F.Cu at (328.4, 192.8)
- added D43: D, Diode_THT:D_DO-35_SOD27_P7.62mm_Horizontal, F.Cu at (328.4, 185.7)
- added D44: D, Diode_THT:D_DO-35_SOD27_P7.62mm_Horizontal, F.Cu at (327.0, 167.9)
- added D45: D, Diode_THT:D_DO-35_SOD27_P7.62mm_Horizontal, F.Cu at (327.0, 175.0)
- added D46: D, Diode_THT:D_DO-35_SOD27_P7.62mm_Horizontal, F.Cu at (266.6, 250.9)
- added D47: D, Diode_THT:D_DO-35_SOD27_P7.62mm_Horizontal, F.Cu at (297.5, 220.1)
- added D48: D, Diode_THT:D_DO-35_SOD27_P7.62mm_Horizontal, F.Cu at (306.9, 208.2)
- added D49: D, Diode_THT:D_DO-35_SOD27_P7.62mm_Horizontal, F.Cu at (337.8, 175.0)
- added D50: D, Diode_THT:D_DO-35_SOD27_P7.62mm_Horizontal, F.Cu at (358.0, 143.1)
- added D51: D, Diode_THT:D_DO-35_SOD27_P7.62mm_Horizontal, F.Cu at (358.0, 139.5)
- added D52: D, Diode_THT:D_DO-35_SOD27_P7.62mm_Horizontal, F.Cu at (306.9, 215.3)
- added D53: D, Diode_THT:D_DO-35_SOD27_P7.62mm_Horizontal, F.Cu at (327.0, 171.5)
- added D54: D, Diode_THT:D_DO-35_SOD27_P7.62mm_Horizontal, F.Cu at (317.7, 203.4)
- added D55: D, Diode_THT:D_DO-35_SOD27_P7.62mm_Horizontal, F.Cu at (348.6, 164.4)
- added D56: D, Diode_THT:D_DO-35_SOD27_P7.62mm_Horizontal, F.Cu at (348.6, 160.8)
- added D57: D, Diode_THT:D_DO-35_SOD27_P7.62mm_Horizontal, F.Cu at (358.0, 146.6)
- added D58: D, Diode_THT:D_DO-35_SOD27_P7.62mm_Horizontal, F.Cu at (328.4, 189.2)
- added D59: D, Diode_THT:D_DO-35_SOD27_P7.62mm_Horizontal, F.Cu at (337.8, 171.5)
- added D60: D, Diode_THT:D_DO-35_SOD27_P7.62mm_Horizontal, F.Cu at (317.7, 192.8)
- added D61: D, Diode_THT:D_DO-35_SOD27_P7.62mm_Horizontal, F.Cu at (306.9, 186.9)
- added D62: D, Diode_THT:D_DO-35_SOD27_P7.62mm_Horizontal, F.Cu at (286.7, 223.7)
- added D63: D, Diode_THT:D_DO-35_SOD27_P7.62mm_Horizontal, F.Cu at (337.8, 167.9)
- added D64: D, Diode_THT:D_DO-35_SOD27_P7.62mm_Horizontal, F.Cu at (266.6, 243.8)
- added D65: D, Diode_THT:D_DO-35_SOD27_P7.62mm_Horizontal, F.Cu at (328.4, 182.1)
- added K42: SW_SPST, Switch_Keyboard_Kailh:SW_Hotswap_Kailh_1.00u, F.Cu at (335.5, 147.8)
- added K43: SW_SPST, Switch_Keyboard_Kailh:SW_Hotswap_Kailh_1.00u, F.Cu at (174.3, 168.0)
- added K44: SW_SPST, Switch_Keyboard_Kailh:SW_Hotswap_Kailh_1.00u, F.Cu at (194.5, 147.8)
- added K45: SW_SPST, Switch_Keyboard_Kailh:SW_Hotswap_Kailh_1.00u, F.Cu at (295.2, 188.1)
- added K46: SW_SPST, Switch_Keyboard_Kailh:SW_Hotswap_Kailh_1.00u, F.Cu at (214.6, 127.7)
- added K47: SW_SPST, Switch_Keyboard_Kailh:SW_Hotswap_Kailh_1.00u, F.Cu at (234.8, 208.3)
- added K48: SW_SPST, Switch_Keyboard_Kailh:SW_Hotswap_Kailh_1.00u, F.Cu at (234.8, 228.4)
- added K49: SW_SPST, Switch_Keyboard_Kailh:SW_Hotswap_Kailh_1.00u, F.Cu at (134.0, 228.4)
- added K50: SW_SPST, Switch_Keyboard_Kailh:SW_Hotswap_Kailh_1.00u, F.Cu at (254.9, 127.7)
- added K51: SW_SPST, Switch_Keyboard_Kailh:SW_Hotswap_Kailh_1.00u, F.Cu at (174.3, 248.6)
- added K52: SW_SPST, Switch_Keyboard_Kailh:SW_Hotswap_Kailh_1.00u, F.Cu at (154.2, 208.3)
- added K53: SW_SPST, Switch_Keyboard_Kailh:SW_Hotswap_Kailh_1.00u, F.Cu at (174.3, 188.1)
- added K54: SW_SPST, Switch_Keyboard_Kailh:SW_Hotswap_Kailh_1.00u, F.Cu at (254.9, 188.1)
- added K55: SW_SPST, Switch_Keyboard_Kailh:SW_Hotswap_Kailh_1.00u, F.Cu at (234.8, 168.0)
- added K56: SW_SPST, Switch_Keyboard_Kailh:SW_Hotswap_Kailh_1.00u, F.Cu at (275.1, 228.4)
- added K57: SW_SPST, Switch_Keyboard_Kailh:SW_Hotswap_Kailh_1.00u, F.Cu at (295.2, 208.3)
- added K58: SW_SPST, Switch_Keyboard_Kailh:SW_Hotswap_Kailh_1.00u, F.Cu at (254.9, 248.6)
- added K59: SW_SPST, Switch_Keyboard_Kailh:SW_Hotswap_Kailh_1.00u, F.Cu at (214.6, 147.8)
- added K60: SW_SPST, Switch_Keyboard_Kailh:SW_Hotswap_Kailh_1.00u, F.Cu at (295.2, 147.8)
- added K61: SW_SPST, Switch_Keyboard_Kailh:SW_Hotswap_Kailh_1.00u, F.Cu at (214.6, 248.6)
- added K62: SW_SPST, Switch_Keyboard_Kailh:SW_Hotswap_Kailh_1.00u, F.Cu at (234.8, 127.7)
- added K63: SW_SPST, Switch_Keyboard_Kailh:SW_Hotswap_Kailh_1.00u, F.Cu at (134.0, 248.6)
- added K64: SW_SPST, Switch_Keyboard_Kailh:SW_Hotswap_Kailh_1.00u, F.Cu at (154.2, 228.4)
- added K65: SW_SPST, Switch_Keyboard_Kailh:SW_Hotswap_Kailh_1.00u, F.Cu at (355.7, 127.7)
- K0, K1, K10, K11, K12, K13, K14, K15, K16, K17, K18, K19, K2, K20, K21, K22, K23, K24, K25, K26, K27, K28, K29, K3, K30, K31, K32, K33, K34, K35, K36, K37, K38, K39, K4, K40, K41, K5, K6, K7, K8, K9: footprint Switch_Keyboard_Cherry_MX:SW_Cherry_MX_PCB_1.00u -> Switch_Keyboard_Kailh:SW_Hotswap_Kailh_1.00u
- moved D14 203.8 mm to (359.3, 160.8)
- moved D21 203.2 mm to (358.0, 157.3)
- moved D15 192.1 mm to (337.8, 178.6)
- moved K26 188.9 mm to (194.5, 248.6)
- moved K13 172.2 mm to (174.3, 228.4)
- moved D24 170.7 mm to (327.0, 178.6)
- moved K19 169.8 mm to (275.1, 208.3)
- moved D17 163.9 mm to (277.4, 240.3)
- moved K38 162.4 mm to (134.0, 127.7)
- moved D31 161.8 mm to (306.9, 197.6)
- moved D29 161.0 mm to (337.8, 164.4)
- moved K27 153.0 mm to (134.0, 168.0)
- moved D40 151.0 mm to (327.0, 163.2)
- moved K41 144.1 mm to (134.0, 208.3)
- moved K25 142.1 mm to (315.4, 168.0)
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
Commit message: Updated Makefile
Parts:
- added D66: D, Diode_SMD:D_SOD-123, F.Cu at (198.8, 184.9)
- added D67: D, Diode_SMD:D_SOD-123, F.Cu at (204.6, 184.9)
- added D68: D, Diode_SMD:D_SOD-123, F.Cu at (210.3, 181.6)
- added D69: D, Diode_SMD:D_SOD-123, F.Cu at (216.1, 181.6)
- added D70: D, Diode_SMD:D_SOD-123, F.Cu at (210.3, 184.9)
- added D71: D, Diode_SMD:D_SOD-123, F.Cu at (187.3, 181.6)
- added D72: D, Diode_SMD:D_SOD-123, F.Cu at (273.6, 181.6)
- added D73: D, Diode_SMD:D_SOD-123, F.Cu at (279.3, 181.6)
- added D74: D, Diode_SMD:D_SOD-123, F.Cu at (216.1, 184.9)
- added D75: D, Diode_SMD:D_SOD-123, F.Cu at (227.6, 181.6)
- added K66: SW_SPST, Switch_Keyboard_Alps_Matias:SW_Alps_Matias_1.00u, F.Cu at (165.8, 169.8)
- added K67: SW_SPST, Switch_Keyboard_Alps_Matias:SW_Alps_Matias_1.00u, F.Cu at (185.9, 169.8)
- added K68: SW_SPST, Switch_Keyboard_Alps_Matias:SW_Alps_Matias_1.00u, F.Cu at (226.2, 89.2)
- added K69: SW_SPST, Switch_Keyboard_Alps_Matias:SW_Alps_Matias_1.00u, F.Cu at (206.1, 109.4)
- added K70: SW_SPST, Switch_Keyboard_Alps_Matias:SW_Alps_Matias_1.00u, F.Cu at (387.4, 48.9)
- added K71: SW_SPST, Switch_Keyboard_Alps_Matias:SW_Alps_Matias_1.00u, F.Cu at (246.4, 48.9)
- added K72: SW_SPST, Switch_Keyboard_Alps_Matias:SW_Alps_Matias_1.00u, F.Cu at (226.2, 69.1)
- added K73: SW_SPST, Switch_Keyboard_Alps_Matias:SW_Alps_Matias_1.00u, F.Cu at (206.1, 149.7)
- added K74: SW_SPST, Switch_Keyboard_Alps_Matias:SW_Alps_Matias_1.00u, F.Cu at (165.8, 48.9)
- added K75: SW_SPST, Switch_Keyboard_Alps_Matias:SW_Alps_Matias_1.00u, F.Cu at (226.2, 129.5)
- D0, D1, D10, D11, D12, D13, D14, D15, D16, D17, D18, D19, D2, D20, D21, D22, D23, D24, D25, D26, D27, D28, D29, D3, D30, D31, D32, D33, D34, D35, D36, D37, D38, D39, D4, D40, D41, D42, D43, D44, D45, D46, D47, D48, D49, D5, D50, D51, D52, D53, D54, D55, D56, D57, D58, D59, D6, D60, D61, D62, D63, D64, D65, D7, D8, D9: footprint Diode_THT:D_DO-35_SOD27_P7.62mm_Horizontal -> Diode_SMD:D_SOD-123
- K0, K1, K10, K11, K12, K13, K14, K15, K16, K17, K18, K19, K2, K20, K21, K22, K23, K24, K25, K26, K27, K28, K29, K3, K30, K31, K32, K33, K34, K35, K36, K37, K38, K39, K4, K40, K41, K42, K43, K44, K45, K46, K47, K48, K49, K5, K50, K51, K52, K53, K54, K55, K56, K57, K58, K59, K6, K60, K61, K62, K63, K64, K65, K7, K8, K9: footprint Switch_Keyboard_Kailh:SW_Hotswap_Kailh_1.00u -> Switch_Keyboard_Alps_Matias:SW_Alps_Matias_1.00u
- moved K38 279.8 mm to (407.6, 69.1)
- moved K13 250.2 mm to (367.3, 69.1)
- moved K51 249.2 mm to (347.1, 69.1)
- moved K4 235.1 mm to (387.4, 69.1)
- moved K26 229.1 mm to (306.8, 48.9)
- moved K32 216.5 mm to (387.4, 89.2)
- moved K52 209.8 mm to (327.0, 89.2)
- moved K14 207.2 mm to (327.0, 48.9)
- moved K58 200.4 mm to (165.8, 69.1)
- moved K27 199.1 mm to (306.8, 69.1)
- moved K33 199.1 mm to (306.8, 89.2)
- moved K1 195.0 mm to (347.1, 89.2)
- moved K63 195.0 mm to (246.4, 89.2)
- moved K64 195.0 mm to (266.5, 69.1)
- moved K31 193.8 mm to (347.1, 129.5)
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